File: WavePad-KiCAD/CM4_GPIO.kicad_sch (KiCad schematic)
At the start: 20 parts, among them J1 Conn_01x03, J2 Conn_02x07_Odd_Even, J3 Conn_01x03, J7 Micro_SD_Card_Det, U18 RT9742GGJ5, U5 74LVC1G07SE-7, U9 74LVC1G07SE-7

Commit message: Worked on PCB
Almost finished the PCB
Parts:
- removed D2: LED Green, LED_SMD:LED_0603_1608Metric, symbol Device:LED
- removed J1, J3: Conn_01x03, Connector_PinHeader_2.54mm:PinHeader_1x03_P2.54mm_Vertical, symbol Connector_Generic:Conn_01x03
- removed J2: Conn_02x07_Odd_Even, Connector_PinHeader_2.54mm:PinHeader_2x07_P2.54mm_Vertical, symbol Connector_Generic:Conn_02x07_Odd_Even
- removed R1: 1k, Resistor_SMD:R_0402_1005Metric, symbol Device:R
- removed TP3: TestPoint, TestPoint:TestPoint_Pad_2.0x2.0mm, symbol Connector:TestPoint
- removed U9: 74LVC1G07SE-7, Package_TO_SOT_SMD:SOT-353_SC-70-5, symbol CM4IO:74LVC1G07_copy
- added TP1: WL_nDis, TestPoint:TestPoint_Pad_2.0x2.0mm, symbol Connector:TestPoint
- added TP2: BT_nDis, TestPoint:TestPoint_Pad_2.0x2.0mm, symbol Connector:TestPoint
- R4, R5: footprint Resistor_SMD:R_0805_2012Metric_Pad1.15x1.40mm_HandSolder -> Resistor_SMD:R_0805_2012Metric
Connections:
- net BT_nDis: now also TP2.1
- net WL_nDis: now also TP1.1
- no-connect marks 7 -> 8
Other:
- note removed: "A button between pins 13-14 can be used to wake up compute module from power down"
- note removed: "Activity LED"
- note removed: "EEPROM write protect = Jumper Pins 3-4"
- note removed: "Force RPIBOOT = Jumper Pins 1-2"
- note removed: "If compute modules is awake RUN_PG will be high so the button doesn't do anything If the compute module is asleep then RUN_PG will be at 0v and so pull global enable low"
- note removed: "Not Fitted headers"
