File: WavePad-KiCAD/CM4IOv5.kicad_pcb (KiCad board)
At the start: 4 copper layers, 27 parts, among them J15 Conn_01x22_Female, J5 USB_C_Receptacle_USB2.0_14P, J7 Micro_SD_Card_Det, J8 Conn_01x22_Female, U1 USBLC6-4SC6, U18 RT9742GGJ5, U5 74LVC1G07SE-7

Commit message: Base OS
Parts:
- removed H1, H2, H3, H4: MountingHole, MountingHole:MountingHole_2.7mm_M2.5
- removed TP1: WL_nDis, TestPoint:TestPoint_Pad_2.0x2.0mm
- removed TP2: BT_nDis, TestPoint:TestPoint_Pad_2.0x2.0mm
- moved D1 27.4 mm to (148.6, 105.8)
- moved R10 27.1 mm to (147.5, 104.0)
- moved U5 26.9 mm to (149.5, 103.2)
- moved TP5 25.7 mm to (148.6, 99.2)
- moved R4 23.9 mm to (156.8, 83.0)
- moved R5 23.9 mm to (154.8, 83.0)
- moved R29 15.3 mm to (142.0, 93.0), turned to 0 degrees
- moved U18 14.4 mm to (142.5, 95.8)
- moved R18 12.4 mm to (141.2, 101.8)
- moved J5 11.9 mm to (162.0, 101.5)
- moved J7 11.6 mm to (133.5, 99.0)
- moved R17 11.4 mm to (142.8, 101.8)
- moved C5 6.58 mm to (142.2, 99.2), turned to 0 degrees
- moved F1 6.51 mm to (162.0, 95.8)
- moved L1 6.23 mm to (161.2, 93.8)
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Routing:
- net GND: track 0.00 -> 125.3 mm, vias 0 -> 67
- net /USB/USB D+: track 0.00 -> 58.7 mm, vias 0 -> 4
- net /USB/USB D-: track 0.00 -> 58.7 mm, vias 0 -> 4
- net /CM4_HighSpeed/CAM_GPIO: track 0.00 -> 54.1 mm, vias 0 -> 2
- net /+3.3v: track 0.00 -> 54.0 mm, vias 0 -> 4
- net /CM4_GPIO (GPIO, SDCARD)/SD_CMD: track 0.00 -> 29.9 mm
- net /CM4_GPIO (GPIO, SDCARD)/SD_DAT2: track 0.00 -> 27.7 mm
- net /CM4_HighSpeed/SCL1: track 0.00 -> 26.5 mm, vias 0 -> 2
- net /CM4_HighSpeed/SDA1: track 0.00 -> 26.4 mm, vias 0 -> 2
- net /CM4_GPIO (GPIO, SDCARD)/SD_DAT1: track 0.00 -> 25.9 mm
- net /CM4_HighSpeed/+3.3v: track 0.00 -> 25.7 mm, vias 0 -> 2
- net /CM4_GPIO (GPIO, SDCARD)/SD_DAT3: track 0.00 -> 25.0 mm
- net /CM4_GPIO (GPIO, SDCARD)/SD_CLK: track 0.00 -> 25.0 mm
- net /CM4_GPIO (GPIO, SDCARD)/SD_DAT0: track 0.00 -> 24.6 mm
- net /CM4_GPIO (GPIO, SDCARD)/Reserved: track 0.00 -> 21.2 mm, vias 0 -> 2
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- added copper zone on B.Cu, net GND
- added copper zone on F.Cu, net GND
Other:
- board outline added: 56.5 x 67.9 mm
- board text added: "PWR_LED"
- board text added: "USB 5V"
- board text added: "WavePad Designed by: Ginobeano Rev: 1"

Commit message: Finish PCB Design
Parts:
- moved R9 49.2 mm to (122.4, 109.4), turned to -90 degrees
- moved U1 46.8 mm to (121.5, 104.7)
- moved J5 45.2 mm to (119.8, 117.7)
- moved F1 38.6 mm to (126.0, 109.6), turned to 180 degrees
- moved L1 37.8 mm to (126.1, 107.6), turned to 0 degrees
- moved TP3 33.5 mm to (126.1, 104.3)
- moved D1 23.4 mm to (131.7, 122.0)
- moved TP5 22.3 mm to (131.8, 113.9), turned to 0 degrees
- moved U5 22.1 mm to (134.9, 119.8), turned to 180 degrees
- moved R10 21.8 mm to (131.8, 119.2), turned to 0 degrees
- moved J7 21.2 mm to (147.3, 115.1), turned to 180 degrees
- moved J8 16.9 mm to (120.5, 57.5)
- moved R4 16.9 mm to (143.6, 93.5), turned to 180 degrees
- moved J15 16.7 mm to (144.9, 57.5)
- moved Module1 15.8 mm to (158.7, 98.4)
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Routing:
- net GND: track 125.3 -> 90.2 mm, vias 67 -> 81
- net /+5v: track 18.2 -> 30.2 mm
- net /CM4_HighSpeed/DSI0_D0_N: track 18.7 -> 8.19 mm, vias 0 -> 2
- net /CM4_HighSpeed/DSI0_D0_P: track 18.4 -> 8.43 mm, vias 0 -> 2
- net /CM4_GPIO (GPIO, SDCARD)/nPWR_LED: track 15.7 -> 24.8 mm
- net /CM4_HighSpeed/DSI0_D1_P: track 17.3 -> 8.27 mm, vias 0 -> 2
- net /CM4_HighSpeed/DSI0_D1_N: track 17.6 -> 8.59 mm, vias 0 -> 2
- net Net-(J7-DET_B): track 13.4 -> 4.63 mm
- net /CM4_GPIO (GPIO, SDCARD)/SD_PWR_ON: track 15.4 -> 6.73 mm, vias 2 -> 0
- net /CM4_GPIO (GPIO, SDCARD)/SD_PWR: track 11.9 -> 20.5 mm, vias 0 -> 2
- net /CM4_GPIO (GPIO, SDCARD)/Reserved: track 21.2 -> 12.8 mm, vias 2 -> 0
- net /+3.3v: track 54.0 -> 46.3 mm, vias 4 -> 6
- net /CM4_HighSpeed/DSI0_C_N: track 16.0 -> 8.53 mm, vias 0 -> 2
- net /CM4_HighSpeed/DSI0_C_P: track 16.0 -> 9.07 mm, vias 0 -> 2
- net Net-(J7-DET_A): track 10.7 -> 4.79 mm, vias 0 -> 2
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Other:
- board size 56.5 x 67.9 mm -> 56.5 x 72.3 mm
- board text added: "CAMERA"
- board text added: "DISPLAY"
- board text added: "WAVEPAD V1.0 Ginobeano"
- board text removed: "Camera"
- board text removed: "Display"
- board text removed: "PWR_LED"
- board text removed: "USB 5V"
- board text removed: "WavePad Designed by: Ginobeano Rev: 1"

Commit message: Specify Serial-Number placement
Other:
- board text added: "WayWayWay"
Changed lines of the file:
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@@
+		)
+	)
+	(gr_text "WayWayWay"
+		(at 155.55 71.3 0)
+		(layer "B.SilkS")
+		(effects
+			(font
+				(size 1 1)
+				(thickness 0.15)
+			)
+			(justify left bottom mirror)
 		)
 	)
